File: placa/Grupo3_Reg_B/Grupo3_Reg_B/Grupo3_Reg_B/RegB.kicad_sch (KiCad schematic)
At the start: 56 parts, among them J1 Conn_02x07_Counter_Clockwise_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, J2 OP295, J3 Conn_01x02_Pin, J4 Conn_01x02_Pin, J5 Conn_01x02_Pin, Q1 BC847BPN, Q10 BS170, Q3 2N2222, Q4 2N2222, Q5 BC547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

Commit message: modificacion de pcb
Parts:
- removed R29: 20, Resistor_THT:R_Axial_DIN0204_L3.6mm_D1.6mm_P7.62mm_Horizontal, symbol Device:R
- R26: value 2,4k -> 2,7k
- R27: value 1,1K -> 1,2K
- R5: value 3,3K -> 3,6K
Connections:
- net GND: now also R27.1
Changed lines of the file:
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@@
 	)
 	(junction
-		(at 173.99 132.08)
+		(at 53.34 162.56)
 		(diameter 0)
 		(color 0 0 0 0)
 	)
 	(junction
-		(at 53.34 162.56)
+		(at 196.85 115.57)
 		(diameter 0)
 		(color 0 0 0 0)
 	)
 	(junction
-		(at 196.85 115.57)
+		(at 173.99 132.08)
 		(diameter 0)
 		(color 0 0 0 0)
@@
 	(wire
 		(pts
+			(xy 173.99 123.19) (xy 173.99 132.08)
+		)
+		(stroke
+			(width 0)
+			(type default)
+		)
+	)
+	(wire
+		(pts
 			(xy 245.11 46.99) (xy 245.11 49.53)
 		)
@@
 	(wire
 		(pts
-			(xy 173.99 132.08) (xy 196.85 132.08)
-		)
-		(stroke
-			(width 0)
-			(type default)
-		)
-	)
-	(wire
-		(pts
 			(xy 135.89 72.39) (xy 135.89 74.93)
 		)
@@
 	(wire
 		(pts
+			(xy 173.99 132.08) (xy 196.85 132.08)
+		)
+		(stroke
+			(width 0)
+			(type default)
+		)
+	)
+	(wire
+		(pts
 			(xy 53.34 170.18) (xy 66.04 170.18)
 		)
@@
 	(wire
 		(pts
-			(xy 173.99 123.19) (xy 173.99 124.46)
-		)
-		(stroke
-			(width 0)
-			(type default)
-		)
-	)
-	(wire
-		(pts
 			(xy 58.42 128.27) (xy 58.42 132.08)
 		)
@@
 			)
 		)
-		(property "Value" "1,1K"
+		(property "Value" "1,2K"
 			(at 176.53 120.6499 0)
 			(effects
@@
 		)
 		(instances
-			(project ""
+			(project "RegB"
 				(path "/58bebdd7-4e1d-4e7a-a1f6-5bcd5ee394de"
 					(reference "J2")
@@
 		)
 		(instances
-			(project "TP_FINAL_555"
+			(project "RegB"
 				(path "/58bebdd7-4e1d-4e7a-a1f6-5bcd5ee394de"
 					(reference "H1")
@@
 			)
 		)
-		(property "Value" "3,3K"
+		(property "Value" "3,6K"
 			(at 199.39 85.0899 0)
 			(effects
@@
 		)
 		(instances
-			(project ""
+			(project "RegB"
 				(path "/58bebdd7-4e1d-4e7a-a1f6-5bcd5ee394de"
 					(reference "C5")
@@
 			)
 		)
-		(property "Value" "2,4k"
+		(property "Value" "2,7k"
 			(at 199.39 109.2199 0)
 			(effects
@@
 		)
 		(instances
-			(project ""
+			(project "RegB"
 				(path "/58bebdd7-4e1d-4e7a-a1f6-5bcd5ee394de"
 					(reference "Q1")
@@
 		)
 		(instances
-			(project ""
+			(project "RegB"
 				(path "/58bebdd7-4e1d-4e7a-a1f6-5bcd5ee394de"
 					(reference "Q1")
@@
 		)
 		(instances
-			(project "TP_FINAL_555"
+			(project "RegB"
 				(path "/58bebdd7-4e1d-4e7a-a1f6-5bcd5ee394de"
 					(reference "H4")
@@
 		)
 		(instances
-			(project ""
-				(path "/58bebdd7-4e1d-4e7a-a1f6-5bcd5ee394de"
-					(reference "J3")
-					(unit 1)
-				)
-			)
-		)
-	)
-	(symbol
-		(lib_id "Device:R")
-		(at 173.99 128.27 180)
-		(unit 1)
-		(exclude_from_sim no)
-		(in_bom yes)
-		(on_board yes)
-		(dnp no)
-		(fields_autoplaced yes)
-		(property "Reference" "R29"
-			(at 176.53 126.9999 0)
-			(effects
-				(font
-					(size 1.27 1.27)
-				)
-				(justify right)
-			)
-		)
-		(property "Value" "20"
-			(at 176.53 129.5399 0)
-			(effects
-				(font
-					(size 1.27 1.27)
-				)
-				(justify right)
-			)
-		)
-		(property "Footprint" "Resistor_THT:R_Axial_DIN0204_L3.6mm_D1.6mm_P7.62mm_Horizontal"
-			(at 175.768 128.27 90)
-			(effects
-				(font
-					(size 1.27 1.27)
-				)
-				(hide yes)
-			)
-		)
-		(property "Datasheet" "~"
-			(at 173.99 128.27 0)
-			(effects
-				(font
-					(size 1.27 1.27)
-				)
-				(hide yes)
-			)
-		)
-		(property "Description" "Resistor"
-			(at 173.99 128.27 0)
-			(effects
-				(font
-					(size 1.27 1.27)
-				)
-				(hide yes)
-			)
-		)
-		(pin "2"
-		)
-		(pin "1"
-		)
-		(instances
 			(project "RegB"
 				(path "/58bebdd7-4e1d-4e7a-a1f6-5bcd5ee394de"
-					(reference "R29")
+					(reference "J3")
 					(unit 1)
 				)
@@
 		)
 		(instances
-			(project "TP_FINAL_555"
+			(project "RegB"
 				(path "/58bebdd7-4e1d-4e7a-a1f6-5bcd5ee394de"
 					(reference "H2")
@@
 		)
 		(instances
-			(project "TP_FINAL_555"
+			(project "RegB"
 				(path "/58bebdd7-4e1d-4e7a-a1f6-5bcd5ee394de"
 					(reference "H3")
@@
 		)
 		(instances
-			(project ""
+			(project "RegB"
 				(path "/58bebdd7-4e1d-4e7a-a1f6-5bcd5ee394de"
 					(reference "Q5")

Commit message: caps de filtro de ruido de linea
Parts:
- added C1, C6: 10u, Capacitor_THT:CP_Radial_D5.0mm_P2.00mm, symbol Device:C
- added C2, C7: 10n, Capacitor_THT:C_Disc_D5.0mm_W2.5mm_P5.00mm, symbol Device:C
Connections:
- net GND: now also C1.2, C2.2, C6.2, C7.2
- net V_sup: now also C6.1, C7.1
- net Vreg: now also C1.1, C2.1
